File: boards/ears/ears.sch (KiCad schematic (older format))
At the start: 5 parts, among them J1 Conn_01x02_Male, U1 AZ1117-3.3, U2 SPX2920T-5.0_TO263, U3 ESP32-WROOM-32D

Commit message: - Ear boards V1
Parts:
- added C1, C3: 0.1uF, Capacitor_SMD:C_0504_1310Metric_Pad0.83x1.28mm_HandSolder, symbol Device:C_Small
- added C2: 10uF, Capacitor_SMD:C_0504_1310Metric_Pad0.83x1.28mm_HandSolder, symbol Device:C_Small
- added C4, C5, C6: 470uF, Capacitor_Tantalum_SMD:CP_EIA-7343-15_Kemet-W_Pad2.25x2.55mm_HandSolder, symbol Device:C_Small
- added D10, D11, D12, D13, D14, D15, D16, D17, D18, D19, D2, D20, D21, D22, D23, D24, D25, D26, D27, D28, D29, D3, D30, D31, D32, D33, D34, D35, D36, D37, D38, D39, D4, D40, D41, D42, D43, D44, D45, D46, D47, D48, D5, D6, D7, D8, D9: WS2812B, LED_SMD:LED_WS2812B_PLCC4_5.0x5.0mm_P3.2mm, symbol LED:WS2812B
- added J2: ESP32-Serial, Connector_PinHeader_1.00mm:PinHeader_1x06_P1.00mm_Horizontal, symbol Connector:Conn_01x06_Male
- added J4: Conn_01x03_Male, Connector_PinHeader_1.00mm:PinHeader_1x03_P1.00mm_Horizontal, symbol Connector:Conn_01x03_Male
- added R1: 10k, Resistor_SMD:R_0603_1608Metric_Pad0.98x0.95mm_HandSolder, symbol Device:R
- added SW1: BOOT_MODE, Button_Switch_SMD:SW_SPST_TL3342, symbol Switch:SW_Push
- added U4: SPX2920T-5.0_TO263, Package_TO_SOT_SMD:TO-263-3_TabPin2, symbol Regulator_Linear:SPX2920T-5.0_TO263
- J1: value Conn_01x02_Male -> Power; footprint Connector_PinHeader_1.00mm:PinHeader_1x02_P1.00mm_Vertical -> Connector_PinHeader_1.00mm:PinHeader_1x02_P1.00mm_Horizontal
Connections:
- net +3V3: now also C2.1, C3.1, R1.1
- net +5V: now also U1.3 (VI), C4.1, C5.1, C6.1, D10.1 (VDD), D11.1 (VDD), D12.1 (VDD), D13.1 (VDD), D14.1 (VDD), D15.1 (VDD), D16.1 (VDD), D17.1 (VDD), D18.1 (VDD), D19.1 (VDD), D2.1 (VDD), D20.1 (VDD), D21.1 (VDD), D22.1 (VDD), D23.1 (VDD), D24.1 (VDD), D25.1 (VDD), D26.1 (VDD), D27.1 (VDD), D28.1 (VDD), D29.1 (VDD), D3.1 (VDD), D30.1 (VDD), D31.1 (VDD), D32.1 (VDD), D33.1 (VDD), D34.1 (VDD), D35.1 (VDD), D36.1 (VDD), D37.1 (VDD), D38.1 (VDD), D39.1 (VDD), D4.1 (VDD), D40.1 (VDD), D41.1 (VDD), D42.1 (VDD), D43.1 (VDD), D44.1 (VDD), D45.1 (VDD), D46.1 (VDD), D47.1 (VDD), D48.1 (VDD), D5.1 (VDD), D6.1 (VDD), D7.1 (VDD), D8.1 (VDD), D9.1 (VDD), J2.3 (Pin_3)
- net GND: now also C1.2, C2.2, C3.2, C4.2, C5.2, C6.2, D10.3 (VSS), D11.3 (VSS), D12.3 (VSS), D13.3 (VSS), D14.3 (VSS), D15.3 (VSS), D16.3 (VSS), D17.3 (VSS), D18.3 (VSS), D19.3 (VSS), D2.3 (VSS), D20.3 (VSS), D21.3 (VSS), D22.3 (VSS), D23.3 (VSS), D24.3 (VSS), D25.3 (VSS), D26.3 (VSS), D27.3 (VSS), D28.3 (VSS), D29.3 (VSS), D3.3 (VSS), D30.3 (VSS), D31.3 (VSS), D32.3 (VSS), D33.3 (VSS), D34.3 (VSS), D35.3 (VSS), D36.3 (VSS), D37.3 (VSS), D38.3 (VSS), D39.3 (VSS), D4.3 (VSS), D40.3 (VSS), D41.3 (VSS), D42.3 (VSS), D43.3 (VSS), D44.3 (VSS), D45.3 (VSS), D46.3 (VSS), D47.3 (VSS), D48.3 (VSS), D5.3 (VSS), D6.3 (VSS), D7.3 (VSS), D8.3 (VSS), D9.3 (VSS), J2.1 (Pin_1), J4.3 (Pin_3), SW1.2, U4.2 (GND)
- net at D1.2 (DOUT): now also D2.4 (DIN)
- net DATA_LED: now reaches D1.4 (DIN), U3.29 (IO5)
- net BOOT_MODE: now reaches U3.25 (IO0)
- net BOOT_MODE: now also SW1.1
- net at U3.3 (EN): now also C1.1, R1.2
- net RXD: now reaches U3.34 (RXD0/IO3)
- net RXD: now also J2.4 (Pin_4)
- net TXD: now reaches U3.35 (TXD0/IO1)
- net TXD: now also J2.5 (Pin_5)
- net V_BATT: now reaches J1.1 (Pin_1), U2.1 (VI)
- net V_BATT: now also U4.1 (VI); no longer U1.3 (VI)
- new net: D2.2 (DOUT), D3.4 (DIN)
- new net: D3.2 (DOUT), D4.4 (DIN)
- new net: D4.2 (DOUT), D5.4 (DIN)
- new net: D5.2 (DOUT), D6.4 (DIN)
- new net: D6.2 (DOUT), D7.4 (DIN)
- new net: D7.2 (DOUT), D8.4 (DIN)
- new net: D8.2 (DOUT), D9.4 (DIN)
- new net: D10.4 (DIN), D9.2 (DOUT)
- new net: D10.2 (DOUT), D11.4 (DIN)
- new net: D11.2 (DOUT), D12.4 (DIN)
- new net: D12.2 (DOUT), D13.4 (DIN)
- new net: D13.2 (DOUT), D14.4 (DIN)
- new net: D14.2 (DOUT), D15.4 (DIN)
- new net: D15.2 (DOUT), D16.4 (DIN)
- new net: D16.2 (DOUT), D17.4 (DIN)
- new net: D17.2 (DOUT), D18.4 (DIN)
- new net: D18.2 (DOUT), D19.4 (DIN)
- new net: D19.2 (DOUT), D20.4 (DIN)
- new net: D20.2 (DOUT), D21.4 (DIN)
- new net: D21.2 (DOUT), D22.4 (DIN)
- new net: D22.2 (DOUT), D23.4 (DIN)
- new net: D23.2 (DOUT), D24.4 (DIN)
- new net: D24.2 (DOUT), D25.4 (DIN)
- new net: D25.2 (DOUT), D26.4 (DIN)
- new net: D26.2 (DOUT), D27.4 (DIN)
- new net: D27.2 (DOUT), D28.4 (DIN)
- new net: D28.2 (DOUT), D29.4 (DIN)
- new net: D29.2 (DOUT), D30.4 (DIN)
- new net: D30.2 (DOUT), D31.4 (DIN)
- new net: D31.2 (DOUT), D32.4 (DIN)
- new net: D32.2 (DOUT), D33.4 (DIN)
- new net: D36.2 (DOUT), D37.4 (DIN)
- new net: D35.2 (DOUT), D36.4 (DIN)
- new net: D34.2 (DOUT), D35.4 (DIN)
- new net: D33.2 (DOUT), D34.4 (DIN)
- new net: D37.2 (DOUT), D38.4 (DIN)
- new net: D38.2 (DOUT), D39.4 (DIN)
- new net: D39.2 (DOUT), D40.4 (DIN)
- new net: D40.2 (DOUT), D41.4 (DIN)
- new net: D41.2 (DOUT), D42.4 (DIN)
- new net: D42.2 (DOUT), D43.4 (DIN)
- new net: D43.2 (DOUT), D44.4 (DIN)
- new net: D44.2 (DOUT), D45.4 (DIN)
- new net: D47.2 (DOUT), D48.4 (DIN)
- new net: D46.2 (DOUT), D47.4 (DIN)
- new net: D45.2 (DOUT), D46.4 (DIN)
- new net 5V_EAR2: J4.1 (Pin_1), U4.3 (VO)
- new net LED_DATA_OUT: D48.2 (DOUT), J4.2 (Pin_2)
Other:
- moved on the sheet: D1, J1, U1, U2, U3
